Commit message: Added drive wheels

File: description/robot.urdf.xacro (robot description, xacro)
@@ -12,4 +12,7 @@
     <material name="blue">
         <color rgba="0.2 0.2 1 1" />
+    </material>
+    <material name="green">
+        <color rgba="0 0.3 0 1" />
     </material>
     <!-- Example link -->
@@ -29,3 +32,31 @@
         </visual>
     </link>
+    <joint name="left_wheel_joint" type="continuous">
+        <parent link="base_link" />
+        <child link="left_wheel" />
+        <origin xyz="0.0 0.175 0.0" rpy="-${pi/2} 0.0 0.0" />
+        <axis xyz="0.0 0.0 1.0" />
+    </joint>
+    <link name="left_wheel">
+        <visual>
+            <geometry>
+                <cylinder radius="0.04" length="0.05" />
+            </geometry>
+            <material name="green" />
+        </visual>
+    </link>
+    <joint name="right_wheel_joint" type="continuous">
+        <parent link="base_link" />
+        <child link="right_wheel" />
+        <origin xyz="0.0 -0.175 0.0" rpy="${pi/2} 0.0 0.0" />
+        <axis xyz="0.0 0.0 -1.0" />
+    </joint>
+    <link name="right_wheel">
+        <visual>
+            <geometry>
+                <cylinder radius="0.04" length="0.05" />
+            </geometry>
+            <material name="green" />
+        </visual>
+    </link>
 </robot>

Commit message: Added caster wheel

File: description/robot.urdf.xacro (robot description, xacro)
@@ -60,3 +60,16 @@
         </visual>
     </link>
+    <joint name="caster_wheel_joint" type="fixed">
+        <origin xyz="0.24 0.0 0.0" rpy="0.0 0.0 0.0" />
+        <parent link="chassis" />
+        <child link="caster_wheel" />
+    </joint>
+    <link name="castor_wheel">
+        <visual>
+            <geometry>
+                <sphere radius="0.05" />
+            </geometry>
+            <material name="white" />
+        </visual>
+    </link>
 </robot>

Commit message: Added collision

File: description/robot.urdf.xacro (robot description, xacro)
@@ -31,4 +31,10 @@
             <material name="black" />
         </visual>
+        <collision>
+            <origin xyz="0.15 0 0.075" />
+            <geometry>
+                <box size="0.3 0.3 0.15" />
+            </geometry>
+        </collision>
     </link>
     <joint name="left_wheel_joint" type="continuous">
@@ -45,4 +51,9 @@
             <material name="green" />
         </visual>
+        <collision>
+            <geometry>
+                <cylinder radius="0.04" length="0.05" />
+            </geometry>
+        </collision>
     </link>
     <joint name="right_wheel_joint" type="continuous">
@@ -59,4 +70,9 @@
             <material name="green" />
         </visual>
+        <collision>
+            <geometry>
+                <cylinder radius="0.04" length="0.05" />
+            </geometry>
+        </collision>
     </link>
     <joint name="caster_wheel_joint" type="fixed">
@@ -65,5 +81,5 @@
         <child link="caster_wheel" />
     </joint>
-    <link name="castor_wheel">
+    <link name="caster_wheel">
         <visual>
             <geometry>
@@ -72,4 +88,9 @@
             <material name="white" />
         </visual>
+        <collision>
+            <geometry>
+                <sphere radius="0.05" />
+            </geometry>
+        </collision>
     </link>
 </robot>

Commit message: Added inertia and inertial_macros.xacro

File: description/robot.urdf.xacro (robot description, xacro)
@@ -1,4 +1,5 @@
 <?xml version="1.0"?>
 <robot xmlns:xacro="http://www.ros.org/wiki/xacro" name="robot">
+    <xacro:include filename="inertial_macros.xacro" />
     <material name="white">
         <color rgba="1 1 1 1" />
@@ -37,4 +38,7 @@
             </geometry>
         </collision>
+        <xacro:inertial_box mass="0.5" x="0.3" y="0.3" z="0.15">
+            <origin xyz="0.15 0 0.075" rpy="0 0 0" />
+        </xacro:inertial_box>
     </link>
     <joint name="left_wheel_joint" type="continuous">
@@ -56,4 +60,7 @@
             </geometry>
         </collision>
+        <xacro:inertial_cylinder mass="0.1" radius="0.04" length="0.05">
+            <origin xyz="0.0 0.0 0.0" rpy="0.0 0.0 0.0" />
+        </xacro:inertial_cylinder>
     </link>
     <joint name="right_wheel_joint" type="continuous">
@@ -75,4 +82,7 @@
             </geometry>
         </collision>
+        <xacro:inertial_cylinder mass="0.1" radius="0.04" length="0.05">
+            <origin xyz="0.0 0.0 0.0" rpy="0.0 0.0 0.0" />
+        </xacro:inertial_cylinder>
     </link>
     <joint name="caster_wheel_joint" type="fixed">
@@ -93,4 +103,7 @@
             </geometry>
         </collision>
+        <xacro:inertial_sphere mass="0.1" radius="0.04">
+            <origin xyz="0.0 0.0 0.0" rpy="0.0 0.0 0.0" />
+        </xacro:inertial_sphere>
     </link>
 </robot>

Commit message: Added gazebo files

File: description/robot.urdf.xacro (robot description, xacro)
@@ -2,4 +2,5 @@
 <robot xmlns:xacro="http://www.ros.org/wiki/xacro" name="robot">
     <xacro:include filename="inertial_macros.xacro" />
+    <xacro:include filename="gazebo_control.xacro" />
     <material name="white">
         <color rgba="1 1 1 1" />
@@ -42,4 +43,7 @@
         </xacro:inertial_box>
     </link>
+    <gazebo reference="chassis">
+        <material>Gazebo/Black</material>
+    </gazebo>
     <joint name="left_wheel_joint" type="continuous">
         <parent link="base_link" />
@@ -64,4 +68,7 @@
         </xacro:inertial_cylinder>
     </link>
+    <gazebo reference="left_wheel">
+        <material>Gazebo/Green</material>
+    </gazebo>
     <joint name="right_wheel_joint" type="continuous">
         <parent link="base_link" />
@@ -86,4 +93,7 @@
         </xacro:inertial_cylinder>
     </link>
+    <gazebo reference="right_wheel">
+        <material>Gazebo/Green</material>
+    </gazebo>
     <joint name="caster_wheel_joint" type="fixed">
         <origin xyz="0.24 0.0 0.0" rpy="0.0 0.0 0.0" />
@@ -107,3 +117,6 @@
         </xacro:inertial_sphere>
     </link>
+    <gazebo reference="caster_wheel">
+        <material>Gazebo/White</material>
+    </gazebo>
 </robot>
